File: ADCS_bdot/ADCS_bdot.kicad_sch (KiCad schematic)
At the start: 0 parts

Commit message: add: components
Changed lines of the file:
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@@
 		)
 		(pin "PWR_IN" input
-			(at 71.12 69.85 180)
+			(at 71.12 68.58 180)
 			(effects
 				(font
