File: ADCS_bdot/Gyroscope.kicad_sch (KiCad schematic)
At the start: 4 parts, among them U1 I3G4250DTR

Commit message: add: a bunch of stuff
Parts:
- added C31, C32: 100n, Capacitor_SMD:C_0603_1608Metric_Pad1.08x0.95mm_HandSolder, symbol Device:C
- added R7: 10R, Resistor_SMD:R_0603_1608Metric_Pad0.98x0.95mm_HandSolder, symbol Device:R
- C29, C30: footprint (none) -> Capacitor_SMD:C_0603_1608Metric_Pad1.08x0.95mm_HandSolder
- R6: footprint (none) -> Resistor_SMD:R_0603_1608Metric_Pad0.98x0.95mm_HandSolder
Connections:
- net GND: now also C31.2, R7.2
- net at U1.14 (PLLFILT): now also C31.1, C32.1
- net SCL: now reaches U1.2 (SCL/SPC)
- net SDA: now reaches U1.3 (SDA/SDI/SDO)
- net SA0: now reaches U1.4 (SDO/SA0)
- net CS_GYRO: now reaches U1.5 (CS)
- net DRDY_GYRO: now reaches U1.6 (DRDY/INT2)
- net INT1_GYRO: now reaches U1.7 (INT1)
- new net: C32.2, R7.1
Other:
- note added: "PLL FILTER"
- note added: "RC Filter"
