File: ADCS_bdot/MCU_STM32F7.kicad_sch (KiCad schematic)
At the start: 30 parts, among them IC1 STM32F746ZGT6, SW1 SW_Push, Y1 ABM3-8.000MHZ-B4Y-T, Y2 CM7V-T1A-32.768kHz-7pF-10PPM-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

Commit message: add: a bunch of stuff
Parts:
- removed C10, C16, C8: 100n, symbol Device:C
- removed C19, C20: 1u, symbol Device:C
- C1, C11, C12, C13, C14, C15, C17, C18, C2, C21, C22, C23, C24, C3, C4, C5, C6, C7, C9: footprint (none) -> Capacitor_SMD:C_0603_1608Metric_Pad1.08x0.95mm_HandSolder
- R1, R2: footprint (none) -> Resistor_SMD:R_0603_1608Metric_Pad0.98x0.95mm_HandSolder
- Y1: footprint (none) -> Footprintlib_adcs_bdot:ABM3
- Y2: footprint (none) -> Footprintlib_adcs_bdot:CM7V32768TBQA020
Other:
- moved on the sheet: C11, C12, C13, C17, C18, C9
