File: ADCS_bdot/Magnetometer.kicad_sch (KiCad schematic)
At the start: 6 parts, among them IC2 IIS2MDCTR

Commit message: add: a bunch of stuff
Parts:
- C25, C26, C27, C28: footprint (none) -> Capacitor_SMD:C_0603_1608Metric_Pad1.08x0.95mm_HandSolder
- R5: footprint (none) -> Resistor_SMD:R_0603_1608Metric_Pad0.98x0.95mm_HandSolder
Connections:
- net SCL: now reaches IC2.1 (SCL/SPC)
- net CS_MAG: now reaches IC2.3 (CS)
- net SDA: now reaches IC2.4 (SDA/SDI/SDO)
- net INT_MAG: now reaches IC2.7 (INT/DRDY)
Other:
- moved on the sheet: C27
Changed lines of the file:
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@@
 	(text "Place close to VDD_IO"
 		(exclude_from_sim no)
-		(at 125.73 149.86 0)
+		(at 135.89 132.08 0)
 		(effects
 			(font
@@
 	(wire
 		(pts
-			(xy 134.62 146.05) (xy 138.43 146.05)
+			(xy 144.78 128.27) (xy 148.59 128.27)
 		)
 		(stroke
@@
 	(wire
 		(pts
+			(xy 113.03 92.71) (xy 116.84 92.71)
+		)
+		(stroke
+			(width 0)
+			(type default)
+		)
+	)
+	(wire
+		(pts
 			(xy 172.72 92.71) (xy 182.88 92.71)
 		)
@@
 	(wire
 		(pts
-			(xy 130.81 158.75) (xy 134.62 158.75)
+			(xy 113.03 97.79) (xy 116.84 97.79)
+		)
+		(stroke
+			(width 0)
+			(type default)
+		)
+	)
+	(wire
+		(pts
+			(xy 140.97 140.97) (xy 144.78 140.97)
 		)
 		(stroke
@@
 	(wire
 		(pts
-			(xy 134.62 148.59) (xy 134.62 146.05)
+			(xy 144.78 130.81) (xy 144.78 128.27)
+		)
+		(stroke
+			(width 0)
+			(type default)
+		)
+	)
+	(wire
+		(pts
+			(xy 113.03 95.25) (xy 116.84 95.25)
 		)
 		(stroke
@@
 	(wire
 		(pts
-			(xy 134.62 158.75) (xy 134.62 156.21)
+			(xy 144.78 140.97) (xy 144.78 138.43)
+		)
+		(stroke
+			(width 0)
+			(type default)
+		)
+	)
+	(wire
+		(pts
+			(xy 113.03 100.33) (xy 116.84 100.33)
 		)
 		(stroke
@@
 			(width 0)
 			(type default)
+		)
+	)
+	(hierarchical_label "INT_MAG"
+		(shape output)
+		(at 113.03 100.33 180)
+		(effects
+			(font
+				(size 1.27 1.27)
+			)
+			(justify right)
+		)
+	)
+	(hierarchical_label "SDA"
+		(shape bidirectional)
+		(at 113.03 97.79 180)
+		(effects
+			(font
+				(size 1.27 1.27)
+			)
+			(justify right)
+		)
+	)
+	(hierarchical_label "SCL"
+		(shape bidirectional)
+		(at 113.03 95.25 180)
+		(effects
+			(font
+				(size 1.27 1.27)
+			)
+			(justify right)
+		)
+	)
+	(hierarchical_label "CS_MAG"
+		(shape input)
+		(at 113.03 92.71 180)
+		(effects
+			(font
+				(size 1.27 1.27)
+			)
+			(justify right)
 		)
 	)
@@
 			)
 		)
-		(property "Footprint" ""
+		(property "Footprint" "Capacitor_SMD:C_0603_1608Metric_Pad1.08x0.95mm_HandSolder"
 			(at 173.6852 109.22 0)
 			(effects
@@
 	(symbol
 		(lib_id "Device:C")
-		(at 134.62 152.4 0)
+		(at 144.78 134.62 0)
 		(unit 1)
 		(exclude_from_sim no)
@@
 		(dnp no)
 		(property "Reference" "C27"
-			(at 137.16 151.13 0)
+			(at 147.32 133.35 0)
 			(effects
 				(font
@@
 		)
 		(property "Value" "100n"
-			(at 137.16 153.67 0)
+			(at 147.32 135.89 0)
 			(effects
 				(font
@@
 			)
 		)
-		(property "Footprint" ""
-			(at 135.5852 156.21 0)
+		(property "Footprint" "Capacitor_SMD:C_0603_1608Metric_Pad1.08x0.95mm_HandSolder"
+			(at 145.7452 138.43 0)
 			(effects
 				(font
@@
 		)
 		(property "Datasheet" "~"
-			(at 134.62 152.4 0)
+			(at 144.78 134.62 0)
 			(effects
 				(font
@@
 		)
 		(property "Description" "Unpolarized capacitor"
-			(at 134.62 152.4 0)
+			(at 144.78 134.62 0)
 			(effects
 				(font
@@
 	(symbol
 		(lib_id "power:+3V3")
-		(at 138.43 146.05 270)
+		(at 148.59 128.27 270)
 		(unit 1)
 		(exclude_from_sim no)
@@
 		(dnp no)
 		(property "Reference" "#PWR022"
-			(at 134.62 146.05 0)
+			(at 144.78 128.27 0)
 			(effects
 				(font
@@
 		)
 		(property "Value" "+3V3"
-			(at 140.97 146.05 90)
+			(at 151.13 128.27 90)
 			(effects
 				(font
@@
 		)
 		(property "Footprint" ""
-			(at 138.43 146.05 0)
+			(at 148.59 128.27 0)
 			(effects
 				(font
@@
 		)
 		(property "Datasheet" ""
-			(at 138.43 146.05 0)
+			(at 148.59 128.27 0)
 			(effects
 				(font
@@
 		)
 		(property "Description" "Power symbol creates a global label with name \"+3V3\""
-			(at 138.43 146.05 0)
+			(at 148.59 128.27 0)
 			(effects
 				(font
@@
 			)
 		)
-		(property "Footprint" ""
+		(property "Footprint" "Capacitor_SMD:C_0603_1608Metric_Pad1.08x0.95mm_HandSolder"
 			(at 107.6452 114.3 0)
 			(effects
@@
 			)
 		)
-		(property "Footprint" ""
+		(property "Footprint" "Capacitor_SMD:C_0603_1608Metric_Pad1.08x0.95mm_HandSolder"
 			(at 183.8452 109.22 0)
 			(effects
@@
 	(symbol
 		(lib_id "power:GND")
-		(at 130.81 158.75 270)
+		(at 140.97 140.97 270)
 		(unit 1)
 		(exclude_from_sim no)
@@
 		(fields_autoplaced yes)
 		(property "Reference" "#PWR021"
-			(at 124.46 158.75 0)
+			(at 134.62 140.97 0)
 			(effects
 				(font
@@
 		)
 		(property "Value" "GND"
-			(at 127 158.7499 90)
+			(at 137.16 140.9699 90)
 			(effects
 				(font
@@
 		)
 		(property "Footprint" ""
-			(at 130.81 158.75 0)
+			(at 140.97 140.97 0)
 			(effects
 				(font
@@
 		)
 		(property "Datasheet" ""
-			(at 130.81 158.75 0)
+			(at 140.97 140.97 0)
 			(effects
 				(font
@@
 		)
 		(property "Description" "Power symbol creates a global label with name \"GND\" , ground"
-			(at 130.81 158.75 0)
+			(at 140.97 140.97 0)
 			(effects
 				(font
@@
 			)
 		)
-		(property "Footprint" ""
+		(property "Footprint" "Resistor_SMD:R_0603_1608Metric_Pad0.98x0.95mm_HandSolder"
 			(at 190.5 94.488 90)
 			(effects
