File: ADCS_bdot/ADCS_bdot.kicad_pcb (KiCad board)
At the start: 4 copper layers, 89.1 x 92.2 mm, 54 parts, among them IC1 STM32F746ZGT6, IC2 IIS2MDCTR, J5 2053380006, J6 5055671081, J7 2053380006, U1 I3G4250DTR, U3 TPSM861253RDXR, Y1 ABM3-8.000MHZ-B4Y-T, Y2 CM7V-T1A-32.768kHz-7pF-10PPM-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

Commit message: add: components
Parts:
- added AC1: SCA3300-D01-1, Footprintlib_adcs_bdot:SCA3300-D01-1, F.Cu at (130.1, 126.1)
- added IC3: DRV8833RTYR, Footprintlib_adcs_bdot:QFN65P400X400X80-17N-D, F.Cu at (140.0, 124.3)
- added IC4: DRV8833RTYR, Footprintlib_adcs_bdot:QFN65P400X400X80-17N-D, F.Cu at (140.0, 131.5)
- added IC5: HMC1001-RC, Footprintlib_adcs_bdot:HMC1001RC, F.Cu at (171.0, 115.2)
- added U2: TMCS1101A3BQDRQ1, Footprintlib_adcs_bdot:SOIC8_D_TEX, F.Cu at (117.9, 123.5)
- added U4: TMCS1101A3BQDRQ1, Footprintlib_adcs_bdot:SOIC8_D_TEX, F.Cu at (117.9, 130.1)
- added U5: TMCS1101A3BQDRQ1, Footprintlib_adcs_bdot:SOIC8_D_TEX, F.Cu at (117.9, 136.8)
- added U6: HMC1002-TR, Footprintlib_adcs_bdot:SOIC20_HNW, F.Cu at (174.2, 124.8)
- moved R8 7.59 mm to (163.3, 124.8)
- moved C8 7.59 mm to (163.3, 122.2)
- moved R9 7.59 mm to (163.3, 127.3)
